File: Brake.kicad_sch (KiCad schematic)
At the start: 140 parts, among them J1 Conn_02x12_Counter_Clockwise, J10 Conn_01x08, J11 Conn_01x08, J12 Conn_02x12_Counter_Clockwise, J13 Conn_01x08, J14 Conn_01x08, J15 Conn_01x08, J16 Conn_01x08, J17 Conn_01x08, J2 Conn_02x12_Counter_Clockwise, J5 Conn_02x12_Counter_Clockwise, J9 Conn_01x08, K1 HEADER_MALE_5X1, K8 HEADER_MALE_5X1, SW1 SW_SPST, SW2 SW_SPST, U1 STM32F103C8Tx, U2 SN65HVD256D, U3 MAX7219, U4 AP2204K-ADJ, U5 AP63200WU, U8 MAX7219CNG, Y1 8M, Y2 32.768k

Commit message: add BSPD pin & CAN
Parts:
- removed C25, C27: 0.1u, Capacitor_SMD:C_0603_1608Metric, symbol Device:C_Small
- removed D1, D10, D11, D12, D13, D14, D15, D16, D17, D18, D19, D2, D20, D21, D22, D23, D24, D25, D26, D27, D28, D29, D3, D30, D31, D32, D33, D34, D35, D36, D37, D38, D39, D4, D40, D41, D42, D43, D44, D45, D46, D47, D48, D49, D5, D50, D51, D52, D53, D54, D55, D56, D57, D58, D59, D6, D60, D61, D62, D63, D64, D7, D8, D9: 0402LED, e-radionica.com footprinti:0402LED, symbol e-radionica.com schematics:0402LED
- removed DS1: TA08-81GWA, TA08-81GWA:DISPLAY_TA08-81GWA, symbol TA08-81GWA:TA08-81GWA
- removed J1, J12, J2, J5: Conn_02x12_Counter_Clockwise, Package_DIP:DIP-24_W7.62mm_Socket, symbol Connector_Generic:Conn_02x12_Counter_Clockwise
- removed K1, K8: HEADER_MALE_5X1, e-radionica.com footprinti:HEADER_MALE_5X1, symbol e-radionica.com schematics:HEADER_MALE_5X1
- removed R10, R12, R14, R16: 9.53k, Resistor_SMD:R_0603_1608Metric, symbol Device:R_Small
- removed U3: MAX7219, MAX7219CNG:DIP762W47P254L3054H457Q24B, symbol Driver_LED:MAX7219
- added C26, C28, C29: 0.1u, Capacitor_SMD:C_0603_1608Metric, symbol Device:C_Small
- added J1: Conn_01x03, Connector_PinHeader_2.54mm:PinHeader_1x03_P2.54mm_Vertical, symbol Connector_Generic:Conn_01x03
- added J3, J4: Conn_01x05, Connector_PinHeader_2.54mm:PinHeader_1x05_P2.54mm_Vertical, symbol Connector_Generic:Conn_01x05
- added JP1: Jumper_2_Open, Connector_PinHeader_2.54mm:PinHeader_1x02_P2.54mm_Vertical, symbol Jumper:Jumper_2_Open
- added R15, R18, R19: 9.53k, Resistor_SMD:R_0603_1608Metric, symbol Device:R_Small
- added U6, U7, U9: MAX7219CNG, Package_DIP:DIP-24_W7.62mm_Socket, symbol MAX7219CNG:MAX7219CNG
- C16, C23, C24: value 0.1u -> 100n
- U8: footprint MAX7219CNG:DIP762W47P254L3054H457Q24B -> Package_DIP:DIP-24_W7.62mm_Socket
Connections:
- net +3V3: now also C24.1, R6.1
- net +5V: now also C26.1, C28.1, C29.1, R15.1, R18.1, R19.1, U6.19 (V+), U7.19 (V+), U9.19 (V+); no longer C16.2, C24.1, R6.2
- net CAN+: now also J1.1 (Pin_1), JP1.1 (A); no longer R2.1
- net CAN-: now also J1.3 (Pin_3)
- net CAN_RX: now also U2.4 (RXD); no longer U2.1 (TXD)
- net CAN_TX: now also U2.1 (TXD); no longer U2.4 (RXD)
- net COL2_0: now also U6.14 (SEG_A)
- net COL2_1: now also U6.16 (SEG_B)
- net COL2_2: now also U6.20 (SEG_C)
- net COL2_3: now also U6.23 (SEG_D)
- net COL2_4: now also U6.21 (SEG_E)
- net COL2_5: now also U6.15 (SEG_F)
- net COL2_6: now also U6.17 (SEG_G)
- net COL2_7: now also U6.22 (SEG_DP)
- net COL3_0: now also U7.14 (SEG_A)
- net COL3_1: now also U7.16 (SEG_B)
- net COL3_2: now also U7.20 (SEG_C)
- net COL3_3: now also U7.23 (SEG_D)
- net COL3_4: now also U7.21 (SEG_E)
- net COL3_5: now also U7.15 (SEG_F)
- net COL3_6: now also U7.17 (SEG_G)
- net COL3_7: now also U7.22 (SEG_DP)
- net COL4_0: now also U9.14 (SEG_A)
- net COL4_1: now also U9.16 (SEG_B)
- net COL4_2: now also U9.20 (SEG_C)
- net COL4_3: now also U9.23 (SEG_D)
- net COL4_4: now also U9.21 (SEG_E)
- net COL4_5: now also U9.15 (SEG_F)
- net COL4_6: now also U9.17 (SEG_G)
- net COL4_7: now also U9.22 (SEG_DP)
- net DIN: now also J3.3 (Pin_3)
- net DOUT1: now also U6.1 (DIN)
- net DOUT2: now also U6.24 (DOUT), U7.1 (DIN)
- net DOUT3: now also U7.24 (DOUT), U9.1 (DIN)
- net DOUT4: now also J4.3 (Pin_3), U9.24 (DOUT)
- net GND: now also C26.2, C28.2, C29.2, J3.2 (Pin_2), J4.2 (Pin_2), U6.4 (GND), U6.9 (GND), U7.4 (GND), U7.9 (GND), U9.4 (GND), U9.9 (GND)
- net LOAD: now also J3.4 (Pin_4), J4.4 (Pin_4), U6.12 (LOAD), U7.12 (LOAD), U9.12 (LOAD)
- net ROW2_0: now also U6.2 (DIG_0)
- net ROW2_1: now also U6.11 (DIG_1)
- net ROW2_2: now also U6.6 (DIG_2)
- net ROW2_3: now also U6.7 (DIG_3)
- net ROW2_4: now also U6.3 (DIG_4)
- net ROW2_5: now also U6.10 (DIG_5)
- net ROW2_6: now also U6.5 (DIG_6)
- net ROW2_7: now also U6.8 (DIG_7)
- net ROW3_0: now also U7.2 (DIG_0)
- net ROW3_1: now also U7.11 (DIG_1)
- net ROW3_2: now also U7.6 (DIG_2)
- net ROW3_3: now also U7.7 (DIG_3)
- net ROW3_4: now also U7.3 (DIG_4)
- net ROW3_5: now also U7.10 (DIG_5)
- net ROW3_6: now also U7.5 (DIG_6)
- net ROW3_7: now also U7.8 (DIG_7)
- net ROW4_0: now also U9.2 (DIG_0)
- net ROW4_1: now also U9.11 (DIG_1)
- net ROW4_2: now also U9.6 (DIG_2)
- net ROW4_3: now also U9.7 (DIG_3)
- net ROW4_4: now also U9.3 (DIG_4)
- net ROW4_5: now also U9.10 (DIG_5)
- net ROW4_6: now also U9.5 (DIG_6)
- net ROW4_7: now also U9.8 (DIG_7)
- net SPI_CLK: now also J3.5 (Pin_5), J4.5 (Pin_5), U6.13 (CLK), U7.13 (CLK), U9.13 (CLK)
- net VDC: now also J3.1 (Pin_1), J4.1 (Pin_1)
- net BSPD_IN: now reaches U1.16 (PA6)
- net BSPD_IN: now also C16.2, R6.2
- new net: R19.2, U9.18 (ISET)
- new net: R15.2, U6.18 (ISET)
- new net: R18.2, U7.18 (ISET)
- new net: JP1.2 (B), R2.1
- no-connect marks 26 -> 25
Other:
- note removed: "MAX7219 DRIVER WITH LEDS"
- moved on the sheet: C1, C2, C3, C31, C4, C5, D65, D66, H1, H2, H3, H4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
